File: src/HardwareDesign/USB-PD-PSU.sch (EAGLE design)
At the start: 108 parts, among them IC1 CYPD3177, IC10 MP2315S, IC11 W25Q128JVPIQ, IC12 CAT24C512HU5IGT3, IC2 MCP6001RT-I/OT, IC3 MCP6001RT-I/OT, IC4 MCP4728, IC5 MCP6001RT-I/OT, IC6 MCP6001RT-I/OT, IC7 MCP6001RT-I/OT, IC8 MCP6001RT-I/OT, SW3 TP, X2 K5A1200015304P

Commit message: finished sch. Review needed
Parts:
- added 3VOFB, 3VOUT, FET_3G1, FET_3G2, FET_3G3, FET_3G4, SW3O, VOUT1: TP, ds_passive:TP
- added C41, C43, C44, C45, C46, C47, C49: 100nF, ds_passive:C-0402
- added C42, C48, C50, C61, C62, C64: 1uF, ds_passive:C-0402
- added C51, C52, C53: 100nF, ds_passive:C0402
- added C54: 33pF, ds_passive:C0402
- added C55: 22uF 25V, ds_passive:C-1206
- added C56, C57: 22uF - 10V, ds_passive:C-1206
- added C58, C60: 1uF, ds_passive:C-0603
- added C59: 100nF 50V, ds_passive:C-0603
- added C63: 10uF 50V, ds_passive:C-0603
- added C65, C66: 10uF, ds_passive:C-0402
- added D4: CHIP-FLAT-R_0603, LED:CHIP-FLAT-R_0603-0.55MM
- added D5: CHIP-FLAT-B_0603, LED:CHIP-FLAT-B_0603-0.55MM
- added D6: SMBJ5929B, Diode:ZENERDO-214AA(SMB)
- added IC13: INA219BIDCNT, ds_ic_peripherals:INA219BIDCNT
- added IC14, IC15: MCP6001RT-I/OT, ds_ic_opa:MCP6001RT
- added IC16: ADC-MCP3008-I/SL, ds_ic_peripherals:ADC-MCP3008-I/SL
- added IC17: MP2315S, ds_ic_vreg:MP2315TSOT23-8
- added L3: 4.2uH, ds_passive:L
- added MOSFET3, MOSFET4: DMP3013SFV, ds_active:DMP3013SFV-7POWERDI3333-8_UX_DIO
- added R17: 0.1R 1%, ds_passive:R2512
- added R19, R20, R23, R24, R25, R26, R31, R33, R35, R45, R47, R48, R51, R52: 10K, ds_passive:R0402
- added R29, R30, R32, R36: 1K, ds_passive:R0402
- added R34: (no value), ds_passive:R0805
- added R37: 499K, ds_passive:R0402
- added R39: 7.5K, ds_passive:R0402
- added R40, R46, R49: 10R, ds_passive:R0402
- added R41: 33K, ds_passive:R0402
- added R42: 40.2K, ds_passive:R0402
- added R43: 12.7K, ds_passive:R0402
- added R44: 100K, ds_passive:R0402
- added R53: 390K, ds_passive:R0402
- added S1, S2: 482024764004, Wurth_Switch_WS-ENTV:482024764004
- added T2, T4: BSS138, ds_active:BSS138
- added U$1: 128X32FOLDED, ds_displays:128X32FOLDED
- C6: value 1uF 50V -> 10uF 50V
Connections:
- removed net VOUT: C5.1, C6.1, C7.1, CON1.1, CON1.3, CON2.1, CON2.3, IC1.VDC_OUT, MOSFET2.D, MOSFET2.D_2, MOSFET2.D_3, MOSFET2.D_4, VOUT.P$1
- new net 3V3_OUT: 3VOUT.P$1, C54.1, C56.1, C57.1, C60.1, L3.2, MOSFET3.S, MOSFET3.S_2, MOSFET3.S_3, R42.1, R45.1
- new net ADC_3VFB: 3VFB.P$1, C27.2, IC16.CH5, R12.2, R13.2, R14.1
- new net ADC_3VOUT: 3VOFB.P$1, C54.2, IC16.CH6, R41.2, R42.2, R43.1
- new net ADC_VBUS: IC16.CH7, R35.2, R36.1
- new net ADC_VOUT: IC16.CH4, R31.2, R32.1
- new net ADC_VREF: C49.1, C50.1, IC16.VREF, R34.1
- new net DSP_RES: R52.2, U$1.RES#
- new net FET_3V_EN: FET_3G1.P$1, IC9.UART0_TX/I2C0_SDA/SPI1_MISO/GPIO12, R46.1, R47.1
- new net FET_G1: C58.2, D6.C, FET_3G3.P$1, MOSFET4.G, R48.2, T4.D
- new net FET_PD_EN: FET_3G4.P$1, IC9.UART1_RTS/I2C1_SCL/SPI1_MOSI/GPIO11, R49.1, R51.1
- new net N$19: D4.C, IC14.-IN, IC14.OUT
- new net N$20: D4.A, R29.2
- new net N$21: D5.C, IC15.-IN, IC15.OUT
- new net N$22: D5.A, R30.2
- new net N$24: IC17.BST, R40.2
- new net N$25: IC17.FB, R41.1
- new net N$26: C53.1, R40.1
- new net N$27: IC17.EN, R37.2
- new net N$28: C52.1, IC17.VCC, R44.1
- new net N$29: IC17.AAM, R39.1, R44.2
- new net N$30: C61.1, U$1.C2+
- new net N$31: C61.2, U$1.C2-
- new net N$32: C62.1, U$1.C1+
- new net N$33: R46.2, T2.G
- new net N$34: C62.2, U$1.C1-
- new net N$35: R53.1, U$1.IREF
- new net N$36: R49.2, T4.G
- new net N$37: C64.1, U$1.VBREF
- new net N$40: C66.1, U$1.VCOMH
- new net RE-I1: R24.2, S2.A
- new net RE-I2: R25.2, S2.B
- new net RE-SWI: C43.1, IC14.+IN, R26.2, S2.1
- new net RE-SWV: C44.1, IC15.+IN, R23.2, S1.1
- new net RE-V1: R19.2, S1.A
- new net RE-V2: R20.2, S1.B
- new net SPI0_CS: IC16.!CS, IC9.UART0_RX/I2C0_SCL/#SPI0_CS/GPIO17, R33.2
- new net SPI0_MISO: IC16.DOUT, IC9.UART0_TX/I2C0_SDA/#SPI0_MISO/GPIO16
- new net SPI0_MOSI: IC16.DIN, IC9.UART0_RTS/I2C1_SCL/#SPI0_MOSI/GPIO19
- new net SPI0_SCK: IC16.CLK, IC9.UART0_CTS/I2C1_SDA/#SPI0_SCK/GPIO18
- new net SW1: C53.2, IC17.SW, L3.1, SW3O.P$1
- new net VOUT-1: C59.1, C63.1, IC13.IN+, MOSFET3.D, MOSFET3.D_2, MOSFET3.D_3, MOSFET3.D_4, MOSFET4.D, MOSFET4.D_2, MOSFET4.D_3, MOSFET4.D_4, R17.1, R31.1, VOUT1.P$1
- new net VOUT-2: C7.1, CON1.1, CON1.3, CON2.1, CON2.3, IC13.IN-, R17.2
- new net VOUT-USB: C5.1, C58.1, C6.1, IC1.VDC_OUT, MOSFET2.D, MOSFET2.D_2, MOSFET2.D_3, MOSFET2.D_4, MOSFET4.S, MOSFET4.S_2, MOSFET4.S_3, R48.1, VOUT.P$1
- net +3V3: now also C41.1, C42.1, C45.1, C46.1, C47.1, C48.1, IC13.VCC, IC14.V+, IC15.V+, IC16.VDD, R19.1, R20.1, R23.1, R24.1, R25.1, R26.1, R33.1, R34.2, R52.1, U$1.VBAT, U$1.VDD
- net FET_G: now also C60.2, FET_3G2.P$1, MOSFET3.G, R45.2, T2.D
- net GND: now also C41.2, C42.2, C43.2, C44.2, C45.2, C46.2, C47.2, C48.2, C49.2, C50.2, C51.2, C52.2, C55.2, C56.2, C57.2, C59.2, C63.2, C64.2, C65.2, C66.2, D6.A, IC13.A0, IC13.A1, IC13.GND, IC14.V-, IC15.V-, IC16.AGND, IC16.DGND, IC17.GND, R32.2, R36.2, R39.2, R43.2, R47.2, R51.2, R53.2, S1.2, S1.COM, S2.2, S2.COM, T2.S, T4.S, U$1.VSS
- net I2C0_SCL: now also IC13.SCL
- net I2C0_SDA: now also IC13.SDA
- net I2C1_SCL: now also U$1.SCL
- net I2C1_SDA: now also U$1.SDA
- net ISINK_C: now also IC16.CH2; no longer IC9.ADC2/GPIO28
- net ISINK_F: now also IC16.CH3; no longer IC9.ADC3/GPIO29
- net N$42: now also C65.1, U$1.VCC; no longer 3VFB.P$1, C27.2, R12.2, R13.2, R14.1
- net N$5: now also MOSFET1.S, MOSFET1.S_2, MOSFET1.S_3; no longer MOSFET1.D, MOSFET1.D_2, MOSFET1.D_3, MOSFET1.D_4
- net VBUS: now also C51.1, C55.1, IC17.IN, MOSFET1.D, MOSFET1.D_2, MOSFET1.D_3, MOSFET1.D_4, R29.1, R30.1, R35.1, R37.1; no longer MOSFET1.S, MOSFET1.S_2, MOSFET1.S_3
- net VBUS_MAX: now also IC16.CH1; no longer IC9.I2C1_SCL/ADC1/GPIO27
- net VBUS_MIN: now also IC16.CH0; no longer IC9.I2C1_SDA/ADC0/GPIO26
Other:
- note added: "0.91 OLED"
- note added: "3.3V"
- note added: "3.3V OUTPUT DC-DC CONVERTER"
- note added: "3.3V-3A MAX OUT"
- note added: "5V/9V/15V/20V-3A MAX OUT"
- note added: "CURRENT ENCODER"
- note added: "CURRENT MEASUREMENT"
- note added: "PSU CONTROL"
- note added: "VOLTAGE ENCODER"
- note added: "VOLTAGE MEASUREMENT"
- note added: "VOUT"
- moved on the sheet: 3VFB, BOOT, C1, C18, C19, C2, C20, C25, C26, C27, C28, C29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

Commit message: PCB design ready
Parts:
- removed C45, C46, C47, C49: 100nF, ds_passive:C-0402
- removed C48, C50: 1uF, ds_passive:C-0402
- removed C59: 100nF 50V, ds_passive:C-0603
- removed C66: 10uF, ds_passive:C-0402
- removed D4: CHIP-FLAT-R_0603, LED:CHIP-FLAT-R_0603-0.55MM
- removed D5: CHIP-FLAT-B_0603, LED:CHIP-FLAT-B_0603-0.55MM
- removed DBG1, DBG2: (no value), ds_con:CON-1X4
- removed IC14, IC15: MCP6001RT-I/OT, ds_ic_opa:MCP6001RT
- removed IC16: ADC-MCP3008-I/SL, ds_ic_peripherals:ADC-MCP3008-I/SL
- removed R29, R30: 1K, ds_passive:R0402
- removed R33, R52: 10K, ds_passive:R0402
- removed R34: (no value), ds_passive:R0805
- removed R53: 390K, ds_passive:R0402
- removed RESET: RS032G05A3SM, BeagleBone_Blue_R3:RS032G05A3SM-SPST-MOMENTARY-SWSMD-1101NE
- removed S1, S2: 482024764004, Wurth_Switch_WS-ENTV:482024764004
- removed U$1: 128X32FOLDED, ds_displays:128X32FOLDED
- removed X2: K5A1200015304P, ds_passive:CRYSTAL
- added C67: 100nF, ds_passive:C-0201
- added CON3, CON4: (no value), ds_con:CON-2X2SMD
- added DISP: 128X64OLED, ds_displays:128X64OLED
- added I-SET, V-SET: 482024764004, Wurth_Switch_WS-ENTV:482024764004
- added RUN, RX, SWCLK, SWDIO, TX: TP, ds_passive:TP
- added X1: 12MHz, Wurth_Quartz Crystals & Oscillators_WE-XTAL:WE-XTAL_CFPX-180_830055295
- BOOT: value RS032G05A3SM -> TP; device BeagleBone_Blue_R3:RS032G05A3SM-SPST-MOMENTARY-SWSMD-1101NE -> ds_passive:TP
- C10, C11, C12, C13, C14, C15, C16, C17, C18, C21, C26, C28, C29, C30, C31, C32, C33, C34, C37, C38, C39, C41, C42, C43, C44, C8, C9: device ds_passive:C-0402 -> ds_passive:C-0201
- C61, C62, C64: value 1uF -> 2.2uF; device ds_passive:C-0402 -> ds_passive:C-0201
- C65: value 10uF -> 2.2uF; device ds_passive:C-0402 -> ds_passive:C-0201
- C7: device ds_passive:C-1206 -> ds_passive:C-0805
- CON1, CON2: device ds_con:CON-2X2 -> ds_con:CON-2X2SMD
- D1, D6: device Diode:ZENERDO-214AA(SMB) -> Diode:ZENERDO-214AC(SMA)
- L1: value 3.3uH -> 3.3uH LQM21PN3R3MGRD; device ds_passive:L -> ds_passive:R0805
- R16, R19, R20, R21, R22, R23, R24, R25, R26, R4, R5, R6, R7, R8: device ds_passive:R0402 -> ds_passive:R0201
- R27: value NC -> 10K; device ds_passive:R0402 -> ds_passive:R0201
- R28: value 4.7K -> (none); device ds_passive:R0402 -> ds_passive:R0201
- renumbered D2 to FAULT, D3 to FLIP
Connections:
- net N$12 renamed MCU_DP_N
- net N$18 renamed MCU_DP_P
- removed net ADC_VREF: C49.1, C50.1, IC16.VREF, R34.1
- removed net N$21: D5.C, IC15.-IN, IC15.OUT
- removed net N$22: D5.A, R30.2
- removed net N$30: C61.1, U$1.C2+
- removed net N$31: C61.2, U$1.C2-
- removed net N$32: C62.1, U$1.C1+
- removed net N$40: C66.1, U$1.VCOMH
- removed net N$42: C65.1, U$1.VCC
- new net FET_G2: C58.2, D6.C, FET_3G3.P$1, MOSFET4.G, R48.2, T4.D
- new net N$12: C61.2, DISP.C2P
- new net N$18: C61.1, DISP.C2N
- net !QSPI_SS: now also BOOT.P$1; no longer BOOT.1
- net +3V3: now also C67.1, DISP.BS1, DISP.VBAT, DISP.VDD, R27.1, R6.1, R7.1; no longer C45.1, C46.1, C47.1, C48.1, IC14.V+, IC15.V+, IC16.VDD, R27.2, R33.1, R34.2, R52.1, U$1.VBAT, U$1.VDD
- net ADC_3VFB: now also IC9.I2C1_SCL/ADC1/GPIO27; no longer IC16.CH5
- net ADC_3VOUT: now also IC9.ADC2/GPIO28; no longer IC16.CH6
- net ADC_VBUS: now also IC9.ADC3/GPIO29; no longer IC16.CH7
- net ADC_VOUT: now also IC9.I2C1_SDA/ADC0/GPIO26; no longer IC16.CH4
- net DSP_RES: now also DISP./RES; no longer R52.2, U$1.RES#
- net FET_G: no longer C60.2, FET_3G2.P$1, MOSFET3.G, R45.2, T2.D
- net FET_G1: now also C60.2, FET_3G2.P$1, MOSFET3.G, R45.2, T2.D; no longer C58.2, D6.C, FET_3G3.P$1, MOSFET4.G, R48.2, T4.D
- net GND: now also C67.2, CON3.2, CON3.4, CON4.2, CON4.4, DISP.BS0, DISP.BS2, DISP.DC/I2C_SA0, DISP.NC(GND)@1, DISP.NC(GND)@2, DISP.VSS, I-SET.2, I-SET.COM, IC12.A0, R28.2, V-SET.2, V-SET.COM, X1.GND; no longer BOOT.2, C45.2, C46.2, C47.2, C48.2, C49.2, C50.2, C59.2, C66.2, DBG1.P$2, DBG1.P$4, DBG2.P$2, DBG2.P$4, IC14.V-, IC15.V-, IC16.AGND, IC16.DGND, R28.1, R53.2, RESET.1, S1.2, S1.COM, S2.2, S2.COM, U$1.VSS, X2.VDD, X2.VSS
- net I2C0_SCL: now also R38.1; no longer R38.3
- net I2C0_SDA: now also R38.2; no longer R38.4
- net I2C1_SCL: now also DISP.D0/SPI_SCLK/I2C_SCK, R38.3; no longer R38.2, U$1.SCL
- net I2C1_SDA: now also DISP.D1/SPI_SDIN/I2C_SDA, DISP.D2/I2C_SDA, R38.4; no longer R38.1, U$1.SDA
- net ISINK_C: no longer IC16.CH2
- net ISINK_F: no longer IC16.CH3
- net N$17: now also RUN.P$1; no longer RESET.2
- net N$19: now also C62.1, DISP.C1P; no longer D4.C, IC14.-IN, IC14.OUT
- net N$20: now also C62.2, DISP.C1N; no longer D4.A, R29.2
- net N$23: now also DISP./CS, R27.2; no longer IC12.A0, R27.1, R28.2
- net N$34: now also DISP.VCOMH, R28.1; no longer C62.2, U$1.C1-
- net N$35: now also C65.1, DISP.VCC; no longer R53.1, U$1.IREF
- net N$37: now also DISP.VLSS; no longer U$1.VBREF
- net N$9: now also X1.2; no longer X2.OUT
- net RE-I1: now also I-SET.A; no longer S2.A
- net RE-I2: now also I-SET.B; no longer S2.B
- net RE-SWI: now also I-SET.1; no longer IC14.+IN, S2.1
- net RE-SWV: now also V-SET.1; no longer IC15.+IN, S1.1
- net RE-V1: now also V-SET.A; no longer S1.A
- net RE-V2: now also V-SET.B; no longer S1.B
- net RP_XI: now also X1.1; no longer X2.CON
- net SPI0_CS: no longer IC16.!CS, R33.2
- net SPI0_MISO: no longer IC16.DOUT
- net SPI0_MOSI: no longer IC16.DIN
- net SPI0_SCK: no longer IC16.CLK
- net SWCLK: now also SWCLK.P$1; no longer DBG2.P$1
- net SWDIO: now also SWDIO.P$1; no longer DBG2.P$3
- net UART0_RX: now also RX.P$1; no longer DBG1.P$1
- net UART0_TX: now also TX.P$1; no longer DBG1.P$3
- net VBUS: no longer R29.1, R30.1, R6.1, R7.1
- net VBUS_MAX: no longer IC16.CH1
- net VBUS_MIN: no longer IC16.CH0
- net VOUT-1: no longer C59.1
- net VOUT-2: now also CON3.1, CON3.3, CON4.1, CON4.3
Other:
- note added: "0.96 OLED"
- note removed: "0.91 OLED"
- note removed: "3.3V"
- note removed: "VOLTAGE MEASUREMENT"
- note removed: "VOUT"
